File: hw/minixpad/minixpad.kicad_pcb (KiCad board)
At the start: 2 copper layers, 9 parts, among them J1 COM-09032, U1 NodeMCU-12K, U2 MicroUSB

Commit message: Revisit board designs
Signed-off-by: Jan Hamal Dvořák <mordae@anilinux.org>
Connections:
- B1 pad 2: BSTART -> BA
- B1 pad 3: BSTART -> BA
- B2 pad 2: BSELECT -> BB
- B2 pad 3: BSELECT -> BB
- B3 pad 2: BA -> BSELECT
- B3 pad 3: BA -> BSELECT
- B4 pad 2: BB -> BSTART
- B4 pad 3: BB -> BSTART
- U1 pad 14: BSELECT -> BB
- U1 pad 20: BB -> BSTART
- U1 pad 25: BA -> BSELECT
- U1 pad 7: BSTART -> BA
Routing:
- net BSELECT: track 26.7 -> 41.7 mm
- net BA: track 40.6 -> 28.0 mm
- net BSTART: track 26.7 -> 35.2 mm
- net BB: track 34.1 -> 28.0 mm
- net +5V: track 32.7 -> 30.2 mm
- net J1V: track 39.8 -> 41.7 mm
- net J1H: track 57.7 -> 55.8 mm
